File: PCB/SmpsShield.kicad_pcb (KiCad board)
At the start: 2 copper layers, 237.3 x 119.3 mm, 99 parts, among them J1 Conn_01x06, J2 Conn_01x06, J3 Barrel_Jack_Switch, J4 Conn_01x02, J5 Conn_01x04, J6 Conn_01x03, Q1 BC548, U1 ROB-14450, U2 LM317_3PinPackage, U3 LM2575-5.0BT

Commit message: 0.1.0 release
Parts:
- removed the C1 at (249.9, 47.7)
- removed the C1 at (168.7, 48.1)
- removed the C2 at (229.7, 38.3)
- removed the C2 at (148.5, 38.7)
- removed the C3 at (220.8, 87.4)
- removed the C3 at (139.6, 87.8)
- removed the C4 at (223.8, 43.6)
- removed the C4 at (142.6, 44.0)
- removed the C5 at (222.4, 47.8)
- removed the C5 at (141.2, 48.2)
- removed the C6 at (219.8, 75.1)
- removed the C6 at (138.6, 75.5)
- removed the C7 at (207.5, 58.3)
- removed the C7 at (126.3, 58.7)
- removed the C8 at (217.2, 147.5)
- removed the C8 at (136.0, 147.9)
- removed the D3 at (214.5, 53.2)
- removed the D3 at (133.3, 53.6)
- removed the D4 at (234.0, 137.0)
- removed the D4 at (152.8, 137.4)
- removed the D5 at (230.6, 43.8)
- removed the D5 at (149.4, 44.2)
- removed the D6 at (223.8, 141.5)
- removed the D6 at (142.6, 141.9)
- removed the D7 at (234.0, 147.5)
- removed the D7 at (152.8, 147.9)
- removed the D8 at (224.2, 79.0)
- removed the D8 at (143.0, 79.4)
- removed the J1 at (241.9, 141.7)
- removed the J1 at (160.7, 142.1)
- removed the J2 at (241.9, 146.9)
- removed the J2 at (160.7, 147.3)
- removed the J3 at (204.7, 138.9)
- removed the J3 at (123.5, 139.3)
- removed the J4 at (254.1, 48.7)
- removed the J4 at (172.9, 49.1)
- removed the J5 at (209.3, 43.6)
- removed the J5 at (128.1, 44.0)
- removed the J6 at (214.4, 139.7)
- removed the J6 at (133.2, 140.1)
- removed the L1 at (242.1, 91.3)
- removed the L1 at (160.9, 91.7)
- removed the Q1 at (236.0, 39.2)
- removed the Q1 at (154.8, 39.6)
- removed the R2 at (216.5, 134.1)
- removed the R2 at (135.3, 134.5)
- removed the R3 at (239.8, 47.8)
- removed the R3 at (158.6, 48.2)
- removed the R4 at (261.3, 55.6)
- removed the R4 at (180.1, 56.0)
- removed the R5 at (250.0, 116.8)
- removed the R5 at (168.8, 117.2)
- removed the R6 at (261.3, 59.9)
- removed the R6 at (180.1, 60.3)
- removed the R7 at (227.8, 87.8)
- removed the R7 at (146.6, 88.2)
- removed the RV1 at (229.2, 58.6)
- removed the RV1 at (148.0, 59.0)
- removed the TB1 at (231.6, 82.9)
- removed the TB1 at (150.4, 83.3)
- removed the U1 at (238.1, 122.6)
- removed the U1 at (156.9, 123.0)
- removed the U2 at (245.2, 38.3)
- removed the U2 at (164.0, 38.7)
- removed the U3 at (233.4, 75.1)
- removed the U3 at (152.2, 75.5)
- moved C2 86.4 mm to (143.9, 40.0)
- moved C3 86.4 mm to (135.0, 89.1)
- moved C4 86.4 mm to (138.0, 45.3)
- moved C6 86.4 mm to (134.0, 76.8)
- moved C7 86.4 mm to (121.7, 60.0)
- moved C8 86.4 mm to (131.4, 149.2)
- moved D5 86.4 mm to (144.8, 45.5)
- moved D6 86.4 mm to (138.0, 143.2)
- moved D8 86.4 mm to (138.4, 80.7)
- moved J3 86.4 mm to (118.9, 140.6)
- moved J4 86.4 mm to (168.3, 50.4)
- moved J5 86.4 mm to (123.5, 45.3)
- moved L1 86.4 mm to (156.3, 93.0)
- moved R3 86.4 mm to (154.0, 49.5)
- moved R4 86.4 mm to (175.5, 57.3)
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Routing:
- net (no net): track 3759.2 -> 0.00 mm, vias 38 -> 0
- removed copper zone on B.Cu, net (none)
Other:
- board size 237.3 x 119.3 mm -> 65.1 x 118.8 mm
