File: PCB/Microcontroller.sch (KiCad schematic (older format))
At the start: 32 parts, among them J20 Conn_02x05_Odd_Even, J3 Conn_02x06_Odd_Even, J702 Conn_01x06, SW1 SW_DPST_x2, SW2 SW_DIP_x02, U13 STM32F407VGTx, Y1 8Mhz

Commit message: Refactor Firmware and implement serial communication
Connections:
- net MOT_R1: now also U13.97 (PE0); no longer U13.98 (PE1)
- net MOT_R2: now also U13.98 (PE1); no longer U13.97 (PE0)
Changed lines of the file:
@@
 Text HLabel 6800 2100 2    50   Input ~ 0
 SENS_B_R
-Text HLabel 4700 3200 0    50   Output ~ 0
+Text HLabel 4700 3100 0    50   Output ~ 0
 MOT_R1
 Text HLabel 4700 3400 0    50   Output ~ 0
@@
 Text HLabel 6800 1400 2    50   Input ~ 0
 SENS_A_L
-Text HLabel 4700 3100 0    50   Output ~ 0
+Text HLabel 4700 3200 0    50   Output ~ 0
 MOT_R2
 Text HLabel 6800 5300 2    50   Output ~ 0
