File: PCB/root.kicad_pcb (KiCad board)
At the start: 2 copper layers, 120 x 100 mm, 127 parts, among them J1 Conn_01x06, J11 Barrel_Jack_Switch, J12 Conn_01x04, J13 Conn_01x04, J15 XT60-M, J16 Conn_01x04, J17 Conn_01x04, J19 Conn_01x03_Male, J2 Conn_01x06, J20 Conn_02x05_Odd_Even, J22 Conn_01x03_Male, J23 Conn_01x03_Male, J24 Conn_01x03_Male, J3 Conn_02x06_Odd_Even, J401 Conn_01x03_Male, J601 USB_B_Mini, J602 Conn_01x04, J603 Conn_01x04, J604 Conn_01x04, J605 Conn_01x06, J606 Conn_01x04, J7 Screw_Terminal_01x02, J702 Conn_01x06, SW1 SW_DPST_x2, SW2 SW_DIP_x02, SW601 SW_DPST_x2, U1 ROB-14450, U10 XL4015, U11 STC3100IST, U13 STM32F407VGTx, U2 GY-91, U4 VND830SPTR-E, U401 MCP16301T-I_CHY, U6 GY-NEO6MV2, U601 USBLC6-2SC6, U602 ESP-07, U603 TLV75533PDBV, U604 MCP2551-I-SN, U7 XL4015, U8 XL4015, U9 XL4015, Y1 8Mhz

Commit message: Refactor Firmware and implement serial communication
Parts:
- removed G***: LOGO, noah_footprint:Noone
- removed REF**: KiCad-Logo2_8mm_SilkScreen, Symbol:KiCad-Logo2_8mm_SilkScreen
- removed REF**: OSHW-Logo2_14.6x12mm_SilkScreen, Symbol:OSHW-Logo2_14.6x12mm_SilkScreen
- removed REF**: WEEE-Logo_8.4x12mm_SilkScreen, Symbol:WEEE-Logo_8.4x12mm_SilkScreen
Connections:
- U1 pad 13: /Microcontroller/MOT_R1 -> /Microcontroller/MOT_R2
- U1 pad 14: /Microcontroller/MOT_R2 -> /Microcontroller/MOT_R1
- U13 pad 97: /Microcontroller/MOT_R2 -> /Microcontroller/MOT_R1
- U13 pad 98: /Microcontroller/MOT_R1 -> /Microcontroller/MOT_R2
Routing:
- net /Microcontroller/MOT_R2: track 86.0 -> 82.9 mm
- net /Microcontroller/MOT_R1: track 82.9 -> 86.0 mm
